Commit message: Correct namespace issues

File: mitsubishi_arm_description/robots/mitsubishi_rv_6sdl.urdf.xacro (robot description, xacro)
@@ -7,9 +7,8 @@
   <xacro:include filename="$(find mitsubishi_arm_description)/urdf/mitsubishi_rv_6sdl_arm.gazebo" />
   <!-- Import Rviz colors -->
-  <xacro:include filename="$(find mitsubishi_arm_description)/urdf/materials.xacro" />
+  <!--<xacro:include filename="$(find mitsubishi_arm_description)/urdf/materials.xacro" />-->
   <!-- ros_control plugin -->
   <gazebo>
     <plugin name="gazebo_ros_control" filename="libgazebo_ros_control.so">
-      <robotNamespace>/mitsubishi_arm</robotNamespace>
       <robotSimType>gazebo_ros_control/DefaultRobotHWSim</robotSimType>
     </plugin>

File: mitsubishi_arm_description/urdf/mitsubishi_rv_6sdl_arm.xacro (robot description, xacro)
@@ -76,5 +76,5 @@
       <visual>
           <geometry>
-              <mesh filename="package://mitsubishi_arm_description/meshes/rv-6s_no1arm.stl" scale="0.001 0.001 0.001"/>
+              <mesh filename="package://mitsubishi_arm_description/meshes/rv-6s_no1arm_col.dae" scale="0.001 0.001 0.001"/>
           </geometry>
           <origin xyz="0 0 0.1" rpy="0 ${-PI/2} 0"/>
