Commit message: Add mesh files

File: mitsubishi_arm_description/urdf/mitsubishi_rv_6sdl_arm.xacro (robot description, xacro)
@@ -3,18 +3,15 @@
   <property name="PI" value="3.1415926535897931" />
   <property name="offset_from_limit" value="5.0" />
+  <property name="joint_velocity" value="5.0" />
   <!-- base_link -->
   <link name="base_link" >
     <visual>
       <geometry>
-	<box size="0.455 .204 .239"/>
+          <mesh filename="package://mitsubishi_arm_description/meshes/rv-6s_base.stl" scale="0.001 0.001 0.001"/>
       </geometry>
-      <origin xyz="-0.1125 0 .1185"/>
-      <material name="orange">
-        <color rgba="1 1 1 1"/>
-      </material>
     </visual>
     <collision>
       <geometry>
-	<box size="0.455 .204 .239"/>
+    <box size="0.455 .204 .239"/>
       </geometry>
       <origin xyz="-0.1125 0 .1185"/>
@@ -24,347 +21,321 @@
       <mass value="0.01"/>
       <inertia
-        ixx="1.0" ixy="0.0" ixz="0.0"
-        iyy="1.0" iyz="0.0"
-        izz="1.0"/>
-    </inertial>
+          ixx="1.0" ixy="0.0" ixz="0.0"
+          iyy="1.0" iyz="0.0"
+          izz="1.0"/>
+  </inertial>
   </link>
   <joint name="j1" type="revolute">
-    <axis xyz="0 0 1"/>
-    <limit effort="1000.0" lower="${(-170+offset_from_limit)*PI/180}" upper="${(170-offset_from_limit)*PI/180}" velocity="0.2"/>
-    <parent link="base_link"/>
-    <child link="shoulder_block"/>
-    <origin xyz="0 0 0.239"/>
-   <dynamics damping="100.0" friction="100.0" />
-  </joint>
-  <!-- shoulder_block -->
-  <link name="shoulder_block">
-    <visual>
-      <geometry>
-	<box size="0.200 .327 .111"/>
-      </geometry>
-      <origin xyz="-.100 0 0.0555"/>
-      <material name="orange">
-        <color rgba="1 1 1 1"/>
-      </material>
-    </visual>
-    <collision>
-      <geometry>
-	<box size="0.200 .327 .111"/>
-      </geometry>
-      <origin xyz="-.100 0 0.0555"/>
-    </collision>
-    <inertial>
-      <origin xyz="0 0 1" rpy="0 0 0"/>
-      <mass value="0.01"/>
-      <inertia
-        ixx="1.0" ixy="0.0" ixz="0.0"
-        iyy="1.0" iyz="0.0"
-        izz="1.0"/>
-    </inertial>
+      <axis xyz="0 0 1"/>
+      <limit effort="1000.0" lower="${(-170+offset_from_limit)*PI/180}" upper="${(170-offset_from_limit)*PI/180}" velocity="${joint_velocity}"/>
+      <parent link="base_link"/>
+      <child link="shoulder"/>
+      <origin xyz="0 0 0.239"/>
+      <dynamics damping="100.0" friction="100.0" />
+  </joint>
+  <!-- shoulder-->
+  <link name="shoulder">
+      <visual>
+          <geometry>
+              <mesh filename="package://mitsubishi_arm_description/meshes/rv-6s_shoulder.stl" scale="0.001 0.001 0.001"/>
+          </geometry>
+          <origin xyz="0 0 0.016"/>
+      </visual>
+      <collision>
+          <geometry>
+              <cylinder length="0.327" radius="0.079"/>
+          </geometry>
+      </collision>
+      <inertial>
+          <origin xyz="0 0 1" rpy="0 0 0"/>
+          <mass value="0.01"/>
+          <inertia
+              ixx="1.0" ixy="0.0" ixz="0.0"
+              iyy="1.0" iyz="0.0"
+              izz="1.0"/>
+      </inertial>
   </link>
   <joint name="j2" type="revolute">
-    <axis xyz="0 0 1"/>
-    <limit effort="1000.0" lower="${-92*PI/180}" upper="${(135-offset_from_limit)*PI/180}" velocity="0.2"/>
-    <parent link="shoulder_block"/>
-    <child link="shoulder"/>
-    <origin xyz="0.079 0 0.111" rpy="1.57079632679 0 3.14159265359"/>
-   <dynamics damping="100.0" friction="100.0" />
-  </joint>
-  <!-- shoulder -->
-  <link name="shoulder">
-    <visual>
-      <geometry>
-	<cylinder length="0.327" radius="0.079"/>
-      </geometry>
-      <origin xyz="0 0 0"/>
-      <material name="orange">
-        <color rgba="1 1 1 1"/>
-      </material>
-    </visual>
-    <collision>
-      <geometry>
-        <cylinder length="0.327" radius="0.079"/>
-      </geometry>
-      <origin xyz="0 0 0"/>
-    </collision>
-    <inertial>
-      <origin xyz="0 0 1" rpy="0 0 0"/>
-      <mass value="0.01"/>
-      <inertia
-        ixx="1.0" ixy="0.0" ixz="0.0"
-        iyy="1.0" iyz="0.0"
-        izz="1.0"/>
-    </inertial>
-  </link>
-  <joint name="fixed_joint_1" type="fixed">
-    <axis xyz="0 0 1"/>
-    <parent link="shoulder"/>
-    <child link="upper_arm"/>
-    <origin xyz="0 0.079 0"/>
-   <dynamics damping="100.0" friction="100.0" />
+      <axis xyz="0 0 1"/>
+      <limit effort="1000.0" lower="${-92*PI/180}" upper="${(135-offset_from_limit)*PI/180}" velocity="${joint_velocity}"/>
+      <parent link="shoulder"/>
+      <child link="upper_arm"/>
+      <origin xyz="0.085 0 0.111" rpy="1.57079632679 0 3.14159265359"/>
+      <dynamics damping="100.0" friction="100.0" />
   </joint>
   <!-- upper_arm -->
   <link name="upper_arm">
-    <visual>
-      <geometry>
-	<box size="0.090 0.222 0.02"/>
-      </geometry>
-      <origin xyz="0 0.111 0.102"/>
-      <material name="orange">
-        <color rgba="1 1 1 1"/>
-      </material>
-    </visual>
-    <collision>
-      <geometry>
-	<box size="0.090 0.222 0.02"/>
-      </geometry>
-      <origin xyz="0 0.111 0.102"/>
-    </collision>
-    <inertial>
-      <origin xyz="0 0 1" rpy="0 0 0"/>
-      <mass value="0.01"/>
-      <inertia
-        ixx="1.0" ixy="0.0" ixz="0.0"
-        iyy="1.0" iyz="0.0"
-        izz="1.0"/>
-    </inertial>
+      <visual>
+          <geometry>
+              <mesh filename="package://mitsubishi_arm_description/meshes/rv-6s_no1arm.stl" scale="0.001 0.001 0.001"/>
+          </geometry>
+          <origin xyz="0 0 0.1"/>
+      </visual>
+      <collision>
+          <geometry>
+              <box size="0.090 0.380 0.02"/>
+          </geometry>
+          <origin xyz="0 0.191 0.102"/>
+      </collision>
+      <collision>
+          <geometry>
+              <cylinder length="0.20" radius="0.079"/>
+          </geometry>
+      </collision>
+      <inertial>
+          <origin xyz="0 0 1" rpy="0 0 0"/>
+          <mass value="0.01"/>
+          <inertia
+              ixx="1.0" ixy="0.0" ixz="0.0"
+              iyy="1.0" iyz="0.0"
+              izz="1.0"/>
+      </inertial>
   </link>
   <joint name="j3" type="revolute">
-    <axis xyz="0 0 1"/>
-    <limit effort="1000.0" lower="${(-129+offset_from_limit)*PI/180}" upper="${(166-offset_from_limit)*PI/180}" velocity="0.2"/>
-    <parent link="upper_arm"/>
-    <child link="elbow"/>
-    <origin xyz="0 0.301 0" rpy="0 0 1.57"/>
-   <dynamics damping="100.0" friction="100.0" />
+      <axis xyz="0 0 1"/>
+      <limit effort="1000.0" lower="${(-129+offset_from_limit)*PI/180}" upper="${(166-offset_from_limit)*PI/180}" velocity="${joint_velocity}"/>
+      <parent link="upper_arm"/>
+      <child link="elbow"/>
+      <origin xyz="0 0.380 0" rpy="0 0 1.57"/>
+      <dynamics damping="100.0" friction="100.0" />
   </joint>
   <!-- elbow -->
   <link name="elbow">
-    <visual>
-      <geometry>
-	<cylinder length="0.327" radius="0.079"/>
-      </geometry>
-      <origin xyz="0 0 0"/>
-      <material name="orange">
-        <color rgba="1 1 1 1"/>
-      </material>
-    </visual>
-    <collision>
-      <geometry>
-        <cylinder length="0.327" radius="0.079"/>
-      </geometry>
-      <origin xyz="0 0 0"/>
-    </collision>
-    <inertial>
-      <origin xyz="0 0 1" rpy="0 0 0"/>
-      <mass value="0.01"/>
-      <inertia
-        ixx="1.0" ixy="0.0" ixz="0.0"
-        iyy="1.0" iyz="0.0"
-        izz="1.0"/>
-    </inertial>
-  </link>
-  <joint name="fixed_joint_2" type="fixed">
-    <parent link="elbow"/>
-    <child link="elbow_block"/>
-    <origin xyz="0 -0.100 0"/>
-   <dynamics damping="100.0" friction="100.0" />
-  </joint>
-  <!-- elbow_block -->
-  <link name="elbow_block">
-    <visual>
-      <geometry>
-	<box size="0.225 .126 .239"/>
-      </geometry>
-      <origin xyz="-0.0275 0 0"/>
-      <material name="orange">
-        <color rgba="1 1 1 1"/>
-      </material>
-    </visual>
-    <collision>
-      <geometry>
-	<box size="0.225 .126 .239"/>
-      </geometry>
-      <origin xyz="-0.0275 0 0"/>
-    </collision>
-    <inertial>
-      <origin xyz="0 0 1" rpy="0 0 0"/>
-      <mass value="0.01"/>
-      <inertia
-        ixx="1.0" ixy="0.0" ixz="0.0"
-        iyy="1.0" iyz="0.0"
-        izz="1.0"/>
-    </inertial>
+      <visual>
+          <geometry>
+              <mesh filename="package://mitsubishi_arm_description/meshes/rv-6s_elbow.stl" scale="0.001 0.001 0.001"/>
+          </geometry>
+          <origin xyz="0 0 0.1" rpy="0 ${-PI/2} ${PI}"/>
+      </visual>
+      <collision>
+          <geometry>
+              <cylinder length="0.20" radius="0.079"/>
+          </geometry>
+          <origin xyz="0 0 0"/>
+      </collision>
+      <collision>
+          <geometry>
+              <box size="0.25 .120 .170"/>
+          </geometry>
+          <origin xyz="0 -0.1 0"/>
+      </collision>
+      <inertial>
+          <origin xyz="0 0 1" rpy="0 0 0"/>
+          <mass value="0.01"/>
+          <inertia
+              ixx="1.0" ixy="0.0" ixz="0.0"
+              iyy="1.0" iyz="0.0"
+              izz="1.0"/>
+      </inertial>
   </link>
   <joint name="j4" type="revolute">
-    <axis xyz="0 0 1"/>
-    <limit effort="1000.0" lower="${(-160+offset_from_limit)*PI/180}" upper="${(160-offset_from_limit)*PI/180}" velocity="0.2"/>
-    <parent link="elbow_block"/>
-    <child link="fore_arm"/>
-    <origin xyz="0.079 0 0"  rpy="0 1.5707963267 0"/>
-   <dynamics damping="100.0" friction="100.0" />
+      <axis xyz="0 0 1"/>
+      <limit effort="1000.0" lower="${(-160+offset_from_limit)*PI/180}" upper="${(160-offset_from_limit)*PI/180}" velocity="${joint_velocity}"/>
+      <parent link="elbow"/>
+      <child link="joint_arm"/>
+      <origin xyz="0.079 -0.1 0"  rpy="0 1.5707963267 0"/>
+      <dynamics damping="100.0" friction="100.0" />
+  </joint>
+  <!-- joint_arm -->
+  <link name="joint_arm">
+      <visual>
+          <geometry>
+              <mesh filename="package://mitsubishi_arm_description/meshes/rv-6s_joint_arm.stl" scale="0.001 0.001 0.001"/>
+          </geometry>
+      </visual>
+      <collision>
+          <geometry>
+              <box size="0.170 .120 .346"/>
+          </geometry>
+          <origin xyz="0 0 0.1815"/>
+      </collision>
+      <inertial>
+          <origin xyz="0 0 1" rpy="0 0 0"/>
+          <mass value="0.01"/>
+          <inertia
+              ixx="1.0" ixy="0.0" ixz="0.0"
+              iyy="1.0" iyz="0.0"
+              izz="1.0"/>
+      </inertial>
+  </link>
+  <joint name="fixed_joint_1" type="fixed">
+      <axis xyz="0 0 1"/>
+      <parent link="joint_arm"/>
+      <child link="fore_arm"/>
+      <origin xyz="0 0 0.127"/>
+      <dynamics damping="100.0" friction="100.0" />
   </joint>
   <!-- fore_arm -->
   <link name="fore_arm">
-    <visual>
-      <geometry>
-	<box size="0.170 .120 .346"/>
-      </geometry>
-      <origin xyz="0 0 0.1815"/>
-      <material name="orange">
-        <color rgba="1 1 1 1"/>
-      </material>
-    </visual>
-    <collision>
-      <geometry>
-	<box size="0.170 .120 .346"/>
-      </geometry>
-      <origin xyz="0 0 0.1815"/>
-    </collision>
-    <inertial>
-      <origin xyz="0 0 1" rpy="0 0 0"/>
-      <mass value="0.01"/>
-      <inertia
-        ixx="1.0" ixy="0.0" ixz="0.0"
-        iyy="1.0" iyz="0.0"
-        izz="1.0"/>
-    </inertial>
+      <visual>
+          <geometry>
+              <mesh filename="package://mitsubishi_arm_description/meshes/rv-6s_no2arm.stl" scale="0.001 0.001 0.001"/>
+          </geometry>
+          <origin rpy="${PI/2} 0 0"/>
+          <material name="blue">
+              <color rgba="0 0 1 1"/>
+          </material>
+      </visual>
+      <collision>
+          <geometry>
+              <box size="0.170 .120 .346"/>
+          </geometry>
+          <origin xyz="0 0 0.1815"/>
+      </collision>
+      <inertial>
+          <origin xyz="0 0 1" rpy="0 0 0"/>
+          <mass value="0.01"/>
+          <inertia
+              ixx="1.0" ixy="0.0" ixz="0.0"
+              iyy="1.0" iyz="0.0"
+              izz="1.0"/>
+      </inertial>
   </link>
   <joint name="j5" type="revolute">
-    <axis xyz="0 0 1"/>
-    <limit effort="1000.0" lower="${(-110+offset_from_limit)*PI/180}" upper="${(110-offset_from_limit)*PI/180}" velocity="0.2"/>
-    <parent link="fore_arm"/>
-    <child link="wrist"/>
-    <origin xyz="0 0 0.346"  rpy="0.0 -1.5707963267 0"/>
-   <dynamics damping="100.0" friction="100.0" />
+      <axis xyz="0 0 1"/>
+      <limit effort="1000.0" lower="${(-110+offset_from_limit)*PI/180}" upper="${(110-offset_from_limit)*PI/180}" velocity="${joint_velocity}"/>
+      <parent link="fore_arm"/>
+      <child link="wrist"/>
+      <origin xyz="0 0 0.215"  rpy="0.0 -1.5707963267 0"/>
+      <dynamics damping="100.0" friction="100.0" />
   </joint>
   <!-- wrist -->
   <link name="wrist">
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
Commit message: Add Force/Torque sensor and magnet link

File: mitsubishi_arm_description/urdf/mitsubishi_rv_6sdl_arm.xacro (robot description, xacro)
@@ -220,48 +220,44 @@
       <limit effort="1000.0" lower="${(-360+offset_from_limit)*PI/180}" upper="${(360-offset_from_limit)*PI/180}" velocity="${joint_velocity}"/>
       <parent link="wrist"/>
-      <!--<child link="torque_sensor"/>-->
-      <child link="end_effector"/>
+      <child link="torque_sensor"/>
       <origin xyz="0.085 0 0"  rpy="0 1.5707963267 0"/>
       <dynamics damping="10.0" friction="100.0" />
   </joint>
-  <!-- torque_sensor -->
-  <!--
-     -<link name="torque_sensor">
-     -  <visual>
-     -   <geometry>
-     -  <cylinder  length="0.065" radius="0.065"/>
-     -    </geometry>
-     -    <origin xyz="0 0 0.0325"/>
-     -    <material name="orange">
-     -      <color rgba="1 1 1 1"/>
-     -    </material>
-     -  </visual>
-     -  <collision>
-     -   <geometry>
-     -  <cylinder  length="0.065" radius="0.065"/>
-     -    </geometry>
-     -    <origin xyz="0 0 0.0325"/>
-     -    <material name="orange">
-     -      <color rgba="1 1 1 1"/>
-     -    </material>
-     -  </collision>
-     -  <inertial>
-     -    <origin xyz="0 0 1" rpy="0 0 0"/>
-     -    <mass value="0.01"/>
-     -    <inertia
-     -      ixx="1.0" ixy="0.0" ixz="0.0"
-     -      iyy="1.0" iyz="0.0"
-     -      izz="1.0"/>
-     -  </inertial>
-     -</link>
-     -->
-  <!--<joint name="torque_sensor_joint" type="fixed">-->
-      <!--  <axis xyz="0 0 1"/>-->
-      <!--  <limit effort="1000.0" lower="${(-360+offset_from_limit)*PI/180}" upper="${(360-offset_from_limit)*PI/180}" velocity="0.2"/>-->
-      <!--  <parent link="torque_sensor"/>-->
-      <!--  <child link="end_effector"/>-->
-      <!--  <origin xyz="0 0 0.065"  rpy="0 0 0"/> [> original is 0.085 but we have the torque sensor...<]-->
-      <!-- <dynamics damping="100.0" friction="100.0" />-->
-      <!--</joint>-->
+  <!--torque_sensor/magnet -->
+  <link name="torque_sensor">
+    <visual>
+     <geometry>
+    <cylinder  length="0.111" radius="0.038"/>
+      </geometry>
+      <origin xyz="0 0 0.0550"/>
+      <material name="orange">
+        <color rgba="1 1 1 1"/>
+      </material>
+    </visual>
+    <collision>
+     <geometry>
+    <cylinder  length="0.0111" radius="0.038"/>
+      </geometry>
+      <origin xyz="0 0 0.0550"/>
+      <material name="orange">
+        <color rgba="1 1 1 1"/>
+      </material>
+    </collision>
+    <inertial>
+      <origin xyz="0 0 1" rpy="0 0 0"/>
+      <mass value="0.01"/>
+      <inertia
+        ixx="1.0" ixy="0.0" ixz="0.0"
+        iyy="1.0" iyz="0.0"
+        izz="1.0"/>
+    </inertial>
+  </link>
+  <joint name="torque_sensor_joint" type="fixed">
+    <axis xyz="0 0 1"/>
+    <parent link="torque_sensor"/>
+    <child link="end_effector"/>
+    <origin xyz="0 0 0.111"  rpy="0 0 0"/>
+    <dynamics damping="100.0" friction="100.0" />
+  </joint>
   <!-- end_effector -->
   <link name="end_effector">
